File: _autosave-keeb.kicad_pcb (KiCad board)
At the start: 2 copper layers, 371 parts, among them J1 AVR-ISP-6, SW1 SW_MEC_5E, SW10 SW_Push, SW11 SW_Push, SW12 SW_Push, SW13 SW_Push, SW14 SW_Push, SW15 SW_Push, SW16 SW_Push, SW17 SW_Push, SW18 SW_Push, SW19 SW_Push, SW2 RotaryEncoder_Switch, SW20 SW_Push, SW21 SW_Push, SW22 SW_Push, SW23 SW_Push, SW24 SW_Push, SW25 SW_Push, SW26 SW_Push, SW27 SW_Push, SW28 SW_Push, SW29 SW_Push, SW3 SW_Push, SW30 SW_Push, SW31 SW_Push, SW32 SW_Push, SW33 SW_Push, SW34 SW_Push, SW35 SW_Push, SW36 SW_Push, SW37 SW_Push, SW38 SW_Push, SW39 SW_Push, SW4 SW_Push, SW40 SW_Push, SW41 SW_Push, SW42 SW_Push, SW43 SW_Push, SW44 SW_Push, SW45 SW_Push, SW46 SW_Push, SW47 SW_Push, SW48 SW_Push, SW49 SW_Push, SW5 SW_Push, SW50 SW_Push, SW51 SW_Push, SW52 SW_Push, SW53 SW_Push, SW54 SW_Push, SW55 SW_Push, SW56 SW_Push, SW57 SW_Push, SW58 SW_Push, SW59 SW_Push, SW6 SW_Push, SW60 SW_Push, SW61 SW_Push, SW62 SW_Push, SW63 SW_Push, SW64 SW_Push, SW65 SW_Push, SW66 SW_Push, SW67 SW_Push, SW68 SW_Push, SW69 SW_Push, SW7 SW_Push, SW70 SW_Push, SW71 SW_Push, SW72 SW_Push, SW73 SW_Push, SW74 SW_Push, SW75 SW_Push, SW76 SW_Push, SW77 SW_Push, SW78 SW_Push, SW79 SW_Push, SW8 SW_Push, SW80 SW_Push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

Commit message: first
Parts:
- moved C1 446.8 mm to (243.1, 395.2)
- moved C10 446.8 mm to (132.3, 408.5)
- moved C100 446.8 mm to (33.4, 370.3)
- moved C11 446.8 mm to (124.2, 402.5)
- moved C12 446.8 mm to (120.2, 375.3)
- moved C13 446.8 mm to (100.9, 373.3)
- moved C14 446.8 mm to (117.2, 396.4)
- moved C15 446.8 mm to (117.6, 384.4)
- moved C16 446.8 mm to (129.0, 399.5)
- moved C17 446.8 mm to (100.9, 376.3)
- moved C2 446.8 mm to (220.9, 376.2)
- moved C22 446.8 mm to (110.6, 376.3)
- moved C23 446.8 mm to (146.7, 410.6)
- moved C29 446.8 mm to (122.4, 384.4)
- moved C30 446.8 mm to (148.3, 400.6)
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