File: _autosave-keeb.kicad_pcb (KiCad board)
At the start: 2 copper layers, 304.8 x 99 mm, 288 parts, among them J1 AVR-ISP-6, SW1 SW_MEC_5E, SW10 SW_Push, SW11 SW_Push, SW12 SW_Push, SW13 SW_Push, SW14 SW_Push, SW15 SW_Push, SW16 SW_Push, SW17 SW_Push, SW18 SW_Push, SW19 SW_Push, SW2 RotaryEncoder_Switch, SW20 SW_Push, SW21 SW_Push, SW22 SW_Push, SW23 SW_Push, SW24 SW_Push, SW25 SW_Push, SW26 SW_Push, SW27 SW_Push, SW28 SW_Push, SW29 SW_Push, SW3 SW_Push, SW30 SW_Push, SW31 SW_Push, SW32 SW_Push, SW33 SW_Push, SW34 SW_Push, SW35 SW_Push, SW36 SW_Push, SW37 SW_Push, SW38 SW_Push, SW39 SW_Push, SW4 SW_Push, SW40 SW_Push, SW41 SW_Push, SW42 SW_Push, SW43 SW_Push, SW44 SW_Push, SW45 SW_Push, SW46 SW_Push, SW47 SW_Push, SW48 SW_Push, SW49 SW_Push, SW5 SW_Push, SW50 SW_Push, SW51 SW_Push, SW52 SW_Push, SW53 SW_Push, SW54 SW_Push, SW55 SW_Push, SW56 SW_Push, SW57 SW_Push, SW58 SW_Push, SW59 SW_Push, SW6 SW_Push, SW60 SW_Push, SW61 SW_Push, SW62 SW_Push, SW63 SW_Push, SW64 SW_Push, SW65 SW_Push, SW66 SW_Push, SW67 SW_Push, SW68 SW_Push, SW7 SW_Push, SW8 SW_Push, SW9 SW_Push, U1 ATmega32U4-A, Y1 16 Mhz XTAL

Commit message: began routing for real
Parts:
- turned D116 to 90 degrees
- turned D138 to 90 degrees
- turned D145 to 90 degrees
Routing:
- net +5V: track 523.0 -> 1087.8 mm, vias 9 -> 12
- net COL4: track 0.00 -> 378.4 mm, vias 0 -> 12
- net ROW1: track 0.00 -> 375.3 mm, vias 0 -> 10
- net ROW0: track 93.8 -> 416.5 mm, vias 4 -> 12
- net GND: track 428.7 -> 748.8 mm, vias 4 -> 6
- net COL8: track 0.00 -> 304.6 mm, vias 0 -> 8
- net COL0: track 78.1 -> 378.7 mm, vias 3 -> 12
- net ROW2: track 0.00 -> 293.5 mm, vias 0 -> 6
- net COL3: track 0.00 -> 278.0 mm, vias 0 -> 11
- net COL2: track 11.0 -> 287.8 mm, vias 1 -> 12
- net COL6: track 0.00 -> 258.1 mm, vias 0 -> 17
- net RE2: track 2.66 -> 250.3 mm, vias 1 -> 5
- net COL5: track 0.00 -> 243.1 mm, vias 0 -> 10
- net COL9: track 3.45 -> 202.3 mm, vias 1 -> 6
- net ROW3: track 0.00 -> 131.1 mm
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