File: rgbsideglow.kicad_sch (KiCad schematic)
At the start: 20 parts

Commit message: first
Parts:
- C100, C91, C92, C93, C94, C95, C96, C97, C98, C99: renamed from C?; footprint (none) -> Capacitor_SMD:C_0805_2012Metric_Pad1.18x1.45mm_HandSolder
- gave numbers to parts that had none: 10
Connections:
- net +5V: now also D84.2 (VSS), D85.2 (VSS), D86.2 (VSS), D87.2 (VSS), D88.2 (VSS), D89.2 (VSS), D90.2 (VSS), D91.2 (VSS), D92.2 (VSS), D93.2 (VSS)
- net D(will decide # when routing): now also D88.1 (DOUT), D93.1 (DOUT)
- net at D93.3 (DIN): now also D92.1 (DOUT)
- net at D88.3 (DIN): now also D87.1 (DOUT)
- net at D87.3 (DIN): now also D86.1 (DOUT)
- net at D89.1 (DOUT): now also D90.3 (DIN)
- net at D86.3 (DIN): now also D85.1 (DOUT)
- net at D92.3 (DIN): now also D91.1 (DOUT)
- net at D91.3 (DIN): now also D90.1 (DOUT)
- net at D84.1 (DOUT): now also D85.3 (DIN)
