File: rufokeeb.kicad_sch (KiCad schematic)
At the start: 165 parts

Commit message: first
Parts:
- added D97: D_Small, symbol Device:D_Small
- gave numbers to parts that had none: 165
Connections:
- net COL14: now also D97.2 (A); no longer SW30.2, SW45.2, SW59.2, SW73.2
- net ROW0: now also SW30.2, SW45.2, SW59.2, SW73.2, D97.1 (K)
