File: keeb.kicad_pcb (KiCad board)
At the start: 2 copper layers, 371 parts, among them J1 AVR-ISP-6, SW1 SW_MEC_5E, SW10 SW_Push, SW11 SW_Push, SW12 SW_Push, SW13 SW_Push, SW14 SW_Push, SW15 SW_Push, SW16 SW_Push, SW17 SW_Push, SW18 SW_Push, SW19 SW_Push, SW2 RotaryEncoder_Switch, SW20 SW_Push, SW21 SW_Push, SW22 SW_Push, SW23 SW_Push, SW24 SW_Push, SW25 SW_Push, SW26 SW_Push, SW27 SW_Push, SW28 SW_Push, SW29 SW_Push, SW3 SW_Push, SW30 SW_Push, SW31 SW_Push, SW32 SW_Push, SW33 SW_Push, SW34 SW_Push, SW35 SW_Push, SW36 SW_Push, SW37 SW_Push, SW38 SW_Push, SW39 SW_Push, SW4 SW_Push, SW40 SW_Push, SW41 SW_Push, SW42 SW_Push, SW43 SW_Push, SW44 SW_Push, SW45 SW_Push, SW46 SW_Push, SW47 SW_Push, SW48 SW_Push, SW49 SW_Push, SW5 SW_Push, SW50 SW_Push, SW51 SW_Push, SW52 SW_Push, SW53 SW_Push, SW54 SW_Push, SW55 SW_Push, SW56 SW_Push, SW57 SW_Push, SW58 SW_Push, SW59 SW_Push, SW6 SW_Push, SW60 SW_Push, SW61 SW_Push, SW62 SW_Push, SW63 SW_Push, SW64 SW_Push, SW65 SW_Push, SW66 SW_Push, SW67 SW_Push, SW68 SW_Push, SW69 SW_Push, SW7 SW_Push, SW70 SW_Push, SW71 SW_Push, SW72 SW_Push, SW73 SW_Push, SW74 SW_Push, SW75 SW_Push, SW76 SW_Push, SW77 SW_Push, SW78 SW_Push, SW79 SW_Push, SW8 SW_Push, SW80 SW_Push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

Commit message: changed to 60 :C
Parts:
- removed C100, C77, C78, C79, C80, C81, C82, C83, C84, C85, C86, C87, C88, C89, C90, C91, C92, C93, C94, C95, C96, C97, C98, C99: 100nF, Capacitor_SMD:C_0805_2012Metric_Pad1.18x1.45mm_HandSolder
- removed D162, D163, D164, D165, D166, D167, D168, D169, D170, D171, D172, D173, D174, D175, D176, D92: D_Small, Diode_SMD:D_SOD-123
- removed D70, D71, D72, D73, D74, D75, D76, D77, D78, D79, D80, D81, D82, D83, D84, D85, D86, D87, D88, D89, D90, D91, D92, D93: SK6812MINI, LED_SMD:LED_SK6812MINI_PLCC4_3.5x3.5mm_P1.75mm
- removed SW70, SW71, SW73, SW74, SW79, SW80, SW81, SW82, SW83, SW84: SW_Push, acheron_MXH:MX100H
- removed SW72: SW_Push, acheron_MXH:MX175H
- removed SW75, SW76, SW77: SW_Push, acheron_MXH:MX125H
- removed SW78: SW_Push, acheron_MXH:MX625HR
- D100, D102, D103, D111, D126, D141, D147, D149, D151: moved to B.Cu
- SW16: footprint acheron_MXH:MX100H -> acheron_MXH:MX200HR
- SW17: footprint acheron_MXH:MX100H -> acheron_MXH:MX150H
- SW30: footprint acheron_MXH:MX200HR -> acheron_MXH:MX150H
- SW32: footprint acheron_MXH:MX150H -> acheron_MXH:MX175H
- SW45: footprint acheron_MXH:MX150H -> acheron_MXH:MX225HR
- SW46: footprint acheron_MXH:MX100H -> acheron_MXH:MX225HR
- SW47: footprint acheron_MXH:MX175H -> acheron_MXH:MX100H
- SW57: footprint acheron_MXH:MX100H -> acheron_MXH:MX175H
- SW59: footprint acheron_MXH:MX225HR -> acheron_MXH:MX100H
- SW60, SW62: footprint acheron_MXH:MX100H -> acheron_MXH:MX125H
- SW61: footprint acheron_MXH:MX225HR -> acheron_MXH:MX125H
- SW63: footprint acheron_MXH:MX100H -> acheron_MXH:MX625HR
- moved USB1 418.5 mm to (27.8, 21.3)
- moved D105 356.0 mm to (59.3, 142.6)
- moved D133 341.0 mm to (82.4, 144.3)
- moved D127 338.8 mm to (81.4, 155.1)
- moved D118 332.3 mm to (88.2, 147.6)
- moved D120 332.0 mm to (69.9, 156.8)
- moved D152 331.6 mm to (105.4, 144.3)
- moved D98 325.7 mm to (111.2, 144.3)
- moved D150 321.8 mm to (70.9, 146.0)
- moved SW46 321.6 mm to (19.1, 92.1)
- moved D136 318.9 mm to (98.7, 155.1)
- moved SW60 313.3 mm to (9.53, 111.1)
- moved D126 313.0 mm to (65.2, 146.0), turned to 180 degrees
- moved D124 311.5 mm to (75.7, 153.5)
- moved D123 310.5 mm to (76.7, 146.0)
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Connections:
- net D14 renamed Net-(D15-Pad1)
- net D29 renamed Net-(D30-Pad1)
- net D44 renamed D45
- net Net-(D16-Pad1) renamed D16
- net Net-(D31-Pad1) renamed D31
- net VCC renamed +5V
- D2 pad 3: RGB -> LED
- D59 pad 1: D58 -> D59
- D69 pad 1: Net-(D69-Pad1) -> unconnected-(D69-Pad1)

Commit message: moved keys/neopixels
Parts:
- removed D161: D_Small, Diode_SMD:D_SOD-123
- removed D69: SK6812MINI, LED_SMD:LED_SK6812MINI_PLCC4_3.5x3.5mm_P1.75mm
- removed SW69: SW_Push, acheron_MXH:MX100H
- C10, C11, C12, C13, C14, C16, C17, C18, C19, C20, C21, C22, C23, C24, C25, C26, C27, C28, C29, C30, C31, C32, C33, C34, C35, C36, C38, C39, C40, C41, C42, C43, C44, C45, C46, C47, C50, C51, C52, C53, C54, C55, C56, C57, C58, C59, C60, C61, C63, C64, C65, C66, C67, C68, C69, C70, C71, C72, C74, C75: moved to F.Cu
- SW44: footprint acheron_MXH:MX100H -> acheron_MXH:MX225HR
- SW45: footprint acheron_MXH:MX225HR -> acheron_MXH:MX100H
- SW64, SW65: footprint acheron_MXH:MX100H -> acheron_MXH:MX125H
- moved D1 227.1 mm to (41.3, 19.8), turned to 0 degrees
- moved D123 218.0 mm to (274.6, 54.8), turned to 90 degrees
- moved D31 208.3 mm to (282.6, 60.3)
- moved D108 204.6 mm to (247.7, 39.6), turned to 90 degrees
- moved D45 197.7 mm to (282.6, 79.4)
- moved D151 197.5 mm to (274.6, 92.9), turned to 90 degrees
- moved D4 196.7 mm to (34.9, 41.3)
- moved D137 195.3 mm to (274.6, 73.8), turned to 90 degrees
- moved D15 192.2 mm to (254.0, 41.3)
- moved D150 192.1 mm to (255.6, 92.9), turned to 90 degrees
- moved D16 191.3 mm to (283.4, 38.1)
- moved D2 187.7 mm to (-3.17, 31.8)
- moved D103 186.1 mm to (273.8, 33.3), turned to 90 degrees
- moved D13 182.6 mm to (206.4, 41.3)
- moved D7 182.1 mm to (92.1, 41.3)
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Other:
- board outline added: 904.9 x 1011.8 mm

Commit message: placed caps first attempt
Parts:
- removed C76: 100nF, Capacitor_SMD:C_0805_2012Metric_Pad1.18x1.45mm_HandSolder
- C10, C11, C12, C13, C14, C16, C17, C18, C19, C20, C21, C22, C23, C24, C25, C26, C27, C28, C29, C30, C31, C32, C33, C34, C35, C36, C38, C39, C40, C41, C42, C43, C44, C45, C46, C47, C50, C51, C52, C53, C54, C55, C56, C57, C58, C59, C60, C61, C63, C64, C65, C66, C67, C68, C69, C70, C71, C72, C74, C75: moved to B.Cu
- SW1: footprint Button_Switch_SMD:SW_MEC_5GSH9 -> Button_Switch_SMD:SW_Push_1P1T_NO_6x6mm_H9.5mm
- moved C11 230.9 mm to (286.5, 79.4), turned to 90 degrees
- moved C30 227.9 mm to (274.6, 39.7), turned to 90 degrees
- moved C40 224.4 mm to (258.0, 41.3), turned to 90 degrees
- moved C20 214.1 mm to (-8.73, 31.8), turned to 90 degrees
- moved C22 204.8 mm to (286.5, 60.3), turned to 90 degrees
- moved C38 195.3 mm to (238.9, 60.3), turned to 90 degrees
- moved C50 188.2 mm to (229.4, 41.3), turned to 90 degrees
- moved C75 186.3 mm to (262.7, 60.6), turned to 90 degrees
- moved C65 184.6 mm to (210.3, 41.3), turned to 90 degrees
- moved C54 182.0 mm to (5.56, 60.3), turned to 90 degrees
- moved C56 177.1 mm to (219.9, 60.3), turned to 90 degrees
- moved C33 175.3 mm to (267.5, 98.4), turned to 90 degrees
- moved C70 174.9 mm to (286.5, 98.4), turned to 90 degrees
- moved C66 169.9 mm to (7.94, 79.4), turned to 90 degrees
- moved C45 168.0 mm to (96.0, 41.3), turned to 90 degrees
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Connections:
- C1 pad 2: +5V -> GND
- C10 pad 1: +5V -> GND
- C11 pad 1: +5V -> GND
- C12 pad 1: +5V -> GND
- C13 pad 1: +5V -> GND
- C14 pad 1: +5V -> GND
- C15 pad 1: +5V -> GND
- C16 pad 1: +5V -> GND
- C17 pad 1: +5V -> GND
- C18 pad 1: +5V -> GND
- C19 pad 1: +5V -> GND
- C2 pad 2: +5V -> GND
- C20 pad 1: +5V -> GND
- C21 pad 1: +5V -> GND
- C22 pad 1: +5V -> GND
- C23 pad 1: +5V -> GND
- C24 pad 1: +5V -> GND
- C25 pad 1: +5V -> GND
- C26 pad 1: +5V -> GND
- C27 pad 1: +5V -> GND
- C28 pad 1: +5V -> GND
- C29 pad 1: +5V -> GND
- C3 pad 2: +5V -> GND
- C30 pad 1: +5V -> GND
- C31 pad 1: +5V -> GND
- C32 pad 1: +5V -> GND
- C33 pad 1: +5V -> GND
- C34 pad 1: +5V -> GND
- C35 pad 1: +5V -> GND
- C36 pad 1: +5V -> GND
- C37 pad 1: +5V -> GND
- C38 pad 1: +5V -> GND
- C39 pad 1: +5V -> GND
- C4 pad 2: +5V -> GND
- C40 pad 1: +5V -> GND
- C41 pad 1: +5V -> GND
- C42 pad 1: +5V -> GND
- C43 pad 1: +5V -> GND
- C44 pad 1: +5V -> GND
- C45 pad 1: +5V -> GND
- C46 pad 1: +5V -> GND
- C47 pad 1: +5V -> GND
- C48 pad 1: +5V -> GND
- C49 pad 1: +5V -> GND
- C5 pad 2: +5V -> GND
- C50 pad 1: +5V -> GND
- C51 pad 1: +5V -> GND
- C52 pad 1: +5V -> GND
- C53 pad 1: +5V -> GND
- C54 pad 1: +5V -> GND
- C55 pad 1: +5V -> GND
- C56 pad 1: +5V -> GND
- C57 pad 1: +5V -> GND
- C58 pad 1: +5V -> GND
- C59 pad 1: +5V -> GND
- C6 pad 2: +5V -> GND
- C60 pad 1: +5V -> GND
- C61 pad 1: +5V -> GND
- C62 pad 1: +5V -> GND
- C63 pad 1: +5V -> GND
- C64 pad 1: +5V -> GND
- C65 pad 1: +5V -> GND
- C66 pad 1: +5V -> GND
- C67 pad 1: +5V -> GND
- C68 pad 1: +5V -> GND
- C69 pad 1: +5V -> GND
- C7 pad 2: +5V -> GND
- C70 pad 1: +5V -> GND
- C71 pad 1: +5V -> GND
- C72 pad 1: +5V -> GND
- C73 pad 1: +5V -> GND
- C74 pad 1: +5V -> GND
- C75 pad 1: +5V -> GND
- C8 pad 2: +5V -> GND
- C9 pad 1: +5V -> GND
- D1 pad 1: +5V -> GND
- D10 pad 2: +5V -> GND
- D11 pad 2: +5V -> GND
- D12 pad 2: +5V -> GND
- D13 pad 2: +5V -> GND
- D14 pad 2: +5V -> GND
- D15 pad 2: +5V -> GND
- D16 pad 2: +5V -> GND
- D17 pad 2: +5V -> GND
- D18 pad 2: +5V -> GND
- D19 pad 2: +5V -> GND
- D2 pad 2: +5V -> GND
- D20 pad 2: +5V -> GND
- D21 pad 2: +5V -> GND
- D22 pad 2: +5V -> GND
- D23 pad 2: +5V -> GND
- D24 pad 2: +5V -> GND
- D25 pad 2: +5V -> GND
- D26 pad 2: +5V -> GND
- D27 pad 2: +5V -> GND
- D28 pad 2: +5V -> GND
- D29 pad 2: +5V -> GND
- D3 pad 2: +5V -> GND
- D30 pad 2: +5V -> GND
- D31 pad 2: +5V -> GND
- D32 pad 2: +5V -> GND
- D33 pad 2: +5V -> GND
- D34 pad 2: +5V -> GND
- D35 pad 2: +5V -> GND
- D36 pad 2: +5V -> GND
- D37 pad 2: +5V -> GND
- D38 pad 2: +5V -> GND
- D39 pad 2: +5V -> GND
- D4 pad 2: +5V -> GND
- D40 pad 2: +5V -> GND
- D41 pad 2: +5V -> GND
- D42 pad 2: +5V -> GND
- D43 pad 2: +5V -> GND
- D44 pad 2: +5V -> GND
- D45 pad 2: +5V -> GND
- D46 pad 2: +5V -> GND
- D47 pad 2: +5V -> GND
- D48 pad 2: +5V -> GND
- D49 pad 2: +5V -> GND
- D5 pad 2: +5V -> GND
- D50 pad 2: +5V -> GND
- D51 pad 2: +5V -> GND
- D52 pad 2: +5V -> GND
- D53 pad 2: +5V -> GND
- D54 pad 2: +5V -> GND
- D55 pad 2: +5V -> GND
- D56 pad 2: +5V -> GND
- D57 pad 2: +5V -> GND
- D58 pad 2: +5V -> GND
- D59 pad 2: +5V -> GND
- D6 pad 2: +5V -> GND
- D60 pad 2: +5V -> GND
- D61 pad 2: +5V -> GND
- D62 pad 2: +5V -> GND
- D63 pad 2: +5V -> GND
- D64 pad 2: +5V -> GND
- D65 pad 2: +5V -> GND
- D66 pad 2: +5V -> GND
- D67 pad 2: +5V -> GND
- D68 pad 1: Net-(D68-Pad1) -> unconnected-(D68-Pad1)
- D68 pad 2: +5V -> GND
- D7 pad 2: +5V -> GND
- D8 pad 2: +5V -> GND
- D9 pad 2: +5V -> GND
- J1 pad 6: +5V -> GND
- R3 pad 1: +5V -> GND
- R4 pad 1: +5V -> GND
- R6 pad 1: +5V -> GND
- SW1 pad 1: +5V -> GND
- SW1 pad 2: +5V -> GND
- SW2 pad C: +5V -> GND
- U1 pad 15: +5V -> GND
- U1 pad 19: ROW7 -> unconnected-(U1-Pad19)
- U1 pad 20: ROW8 -> unconnected-(U1-Pad20)
- U1 pad 23: +5V -> GND
- U1 pad 35: +5V -> GND
- U1 pad 43: +5V -> GND
- U1 pad 5: +5V -> GND
- USB1 pad 1: +5V -> GND
- USB1 pad 12: +5V -> GND
- USB1 pad 13: +5V -> GND
- Y1 pad 2: +5V -> GND
- Y1 pad 4: +5V -> GND
