File: keeb.kicad_pcb (KiCad board)
At the start: 2 copper layers, 304.8 x 98.1 mm, 288 parts, among them J1 AVR-ISP-6, SW1 SW_MEC_5E, SW10 SW_Push, SW11 SW_Push, SW12 SW_Push, SW13 SW_Push, SW14 SW_Push, SW15 SW_Push, SW16 SW_Push, SW17 SW_Push, SW18 SW_Push, SW19 SW_Push, SW2 RotaryEncoder_Switch, SW20 SW_Push, SW21 SW_Push, SW22 SW_Push, SW23 SW_Push, SW24 SW_Push, SW25 SW_Push, SW26 SW_Push, SW27 SW_Push, SW28 SW_Push, SW29 SW_Push, SW3 SW_Push, SW30 SW_Push, SW31 SW_Push, SW32 SW_Push, SW33 SW_Push, SW34 SW_Push, SW35 SW_Push, SW36 SW_Push, SW37 SW_Push, SW38 SW_Push, SW39 SW_Push, SW4 SW_Push, SW40 SW_Push, SW41 SW_Push, SW42 SW_Push, SW43 SW_Push, SW44 SW_Push, SW45 SW_Push, SW46 SW_Push, SW47 SW_Push, SW48 SW_Push, SW49 SW_Push, SW5 SW_Push, SW50 SW_Push, SW51 SW_Push, SW52 SW_Push, SW53 SW_Push, SW54 SW_Push, SW55 SW_Push, SW56 SW_Push, SW57 SW_Push, SW58 SW_Push, SW59 SW_Push, SW6 SW_Push, SW60 SW_Push, SW61 SW_Push, SW62 SW_Push, SW63 SW_Push, SW64 SW_Push, SW65 SW_Push, SW66 SW_Push, SW67 SW_Push, SW68 SW_Push, SW7 SW_Push, SW8 SW_Push, SW9 SW_Push, U1 ATmega32U4-A, Y1 16 Mhz XTAL

Commit message: fked up LEDs :C
Parts:
- D10, D11, D12, D13, D14, D15, D16, D17, D18, D19, D20, D21, D22, D23, D24, D25, D26, D27, D28, D29, D3, D30, D31, D32, D33, D34, D35, D36, D37, D38, D39, D4, D40, D41, D42, D43, D44, D45, D46, D47, D48, D49, D5, D50, D51, D52, D53, D54, D55, D56, D57, D58, D59, D6, D60, D61, D62, D63, D64, D65, D66, D67, D68, D7, D8, D9: footprint LED_SMD:LED_SK6812MINI_PLCC4_3.5x3.5mm_P1.75mm -> reverse:MX_SK6812MINI-E_REV
- D2: footprint LED_SMD:LED_SK6812MINI_PLCC4_3.5x3.5mm_P1.75mm -> reverse:MX_SK6812MINI-E_REV; moved to F.Cu
- SW16: footprint acheron_MXH:MX200H -> acheron_MXH:MX200HR
- moved D2 5.06 mm to (71.2, 71.1), turned to 0 degrees
Routing:
- net GND: track 101.6 -> 4165.5 mm, vias 8 -> 246
- net COL1: track 729.4 -> 0.00 mm, vias 36 -> 0
- net COL3: track 574.2 -> 0.00 mm, vias 41 -> 0
- net COL6: track 551.7 -> 0.00 mm, vias 32 -> 0
- net COL8: track 522.3 -> 0.00 mm, vias 38 -> 0
- net COL2: track 515.3 -> 0.00 mm, vias 27 -> 0
- net COL0: track 502.9 -> 0.00 mm, vias 30 -> 0
- net COL7: track 509.7 -> 987.0 mm, vias 36 -> 64
- net D59: track 477.4 -> 0.00 mm, vias 28 -> 0
- net COL9: track 471.0 -> 0.00 mm, vias 24 -> 0
- net Net-(D39-Pad1): track 16.4 -> 462.7 mm, vias 0 -> 18
- net D31: track 446.3 -> 0.00 mm, vias 18 -> 0
- net COL5: track 500.6 -> 859.1 mm, vias 34 -> 46
- net RE1: track 358.5 -> 0.00 mm, vias 12 -> 0
- net LED: track 186.4 -> 12.2 mm, vias 10 -> 1
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
Commit message: replaced LED's in appropriate places
Parts:
- D10, D11, D12, D13, D14, D15, D16, D17, D18, D19, D20, D21, D22, D23, D24, D25, D26, D27, D28, D29, D3, D30, D31, D32, D33, D34, D35, D36, D37, D38, D39, D4, D40, D41, D42, D43, D44, D45, D46, D47, D48, D49, D5, D50, D51, D52, D53, D54, D55, D56, D57, D58, D59, D6, D60, D61, D62, D63, D64, D65, D66, D67, D68, D7, D8, D9: moved to F.Cu
- moved D2 9.82 mm to (71.4, 81.0), turned to 180 degrees
- moved D46 6.47 mm to (85.7, 138.1), turned to 0 degrees
- moved D5 5.50 mm to (128.6, 81.0), turned to 0 degrees
- moved D48 5.33 mm to (133.4, 138.1), turned to 0 degrees
- moved D50 5.25 mm to (171.4, 138.1), turned to 0 degrees
- moved D33 5.24 mm to (104.8, 119.1), turned to 0 degrees
- moved D66 5.24 mm to (319.1, 157.2), turned to 0 degrees
- moved D67 5.24 mm to (338.1, 157.2), turned to 0 degrees
- moved D68 5.24 mm to (357.2, 157.2), turned to 0 degrees
- moved D51 5.24 mm to (190.5, 138.1), turned to 0 degrees
- moved D52 5.22 mm to (209.6, 138.1), turned to 0 degrees
- moved D20 5.09 mm to (138.1, 100.0), turned to 0 degrees
- moved D38 5.07 mm to (200.0, 119.1), turned to 0 degrees
- moved D42 5.07 mm to (276.2, 119.1), turned to 0 degrees
- moved D49 4.97 mm to (152.4, 138.1), turned to 0 degrees
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Routing:
- net GND: track 4165.5 -> 1031.0 mm, vias 246 -> 51
- net COL1: track 0.00 -> 729.4 mm, vias 0 -> 36
- net +5V: track 638.5 -> 1275.3 mm, vias 79 -> 108
- net COL6: track 0.00 -> 551.7 mm, vias 0 -> 32
- net COL8: track 0.00 -> 522.3 mm, vias 0 -> 38
- net COL2: track 0.00 -> 515.3 mm, vias 0 -> 27
- net COL0: track 0.00 -> 502.9 mm, vias 0 -> 30
- net COL7: track 987.0 -> 509.7 mm, vias 64 -> 36
- net COL9: track 0.00 -> 471.0 mm, vias 0 -> 24
- net Net-(D37-Pad1): track 16.5 -> 477.4 mm, vias 0 -> 28
- net D16: track 379.1 -> 0.00 mm, vias 26 -> 0
- net COL5: track 859.1 -> 500.6 mm, vias 46 -> 34
- net RE1: track 0.00 -> 358.5 mm, vias 0 -> 12
- net LED: track 12.2 -> 179.4 mm, vias 1 -> 9
- net MISO: track 125.8 -> 59.6 mm, vias 8 -> 3
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