File: keeb.kicad_pcb (KiCad board)
At the start: 2 copper layers, 304.8 x 98.1 mm, 286 parts, among them J1 AVR-ISP-6, SW1 SW_MEC_5E, SW10 SW_Push, SW11 SW_Push, SW12 SW_Push, SW13 SW_Push, SW14 SW_Push, SW15 SW_Push, SW16 SW_Push, SW17 SW_Push, SW18 SW_Push, SW19 SW_Push, SW2 RotaryEncoder_Switch, SW20 SW_Push, SW21 SW_Push, SW22 SW_Push, SW23 SW_Push, SW24 SW_Push, SW25 SW_Push, SW26 SW_Push, SW27 SW_Push, SW28 SW_Push, SW29 SW_Push, SW3 SW_Push, SW30 SW_Push, SW31 SW_Push, SW32 SW_Push, SW33 SW_Push, SW34 SW_Push, SW35 SW_Push, SW36 SW_Push, SW37 SW_Push, SW38 SW_Push, SW39 SW_Push, SW4 SW_Push, SW40 SW_Push, SW41 SW_Push, SW42 SW_Push, SW43 SW_Push, SW44 SW_Push, SW45 SW_Push, SW46 SW_Push, SW47 SW_Push, SW48 SW_Push, SW49 SW_Push, SW5 SW_Push, SW50 SW_Push, SW51 SW_Push, SW52 SW_Push, SW53 SW_Push, SW54 SW_Push, SW55 SW_Push, SW56 SW_Push, SW57 SW_Push, SW58 SW_Push, SW59 SW_Push, SW6 SW_Push, SW60 SW_Push, SW61 SW_Push, SW62 SW_Push, SW63 SW_Push, SW64 SW_Push, SW65 SW_Push, SW66 SW_Push, SW67 SW_Push, SW68 SW_Push, SW7 SW_Push, SW8 SW_Push, SW9 SW_Push, U1 ATmega32U4-A, Y1 16 Mhz XTAL

Commit message: removed cap labels
Parts:
- moved C9 1.70 mm to (115.0, 161.5)
- moved C62 1.51 mm to (91.5, 161.5)
- moved C64 0.80 mm to (171.1, 104.0)
- moved C25 0.78 mm to (187.3, 161.5)
- moved C41 0.72 mm to (68.4, 161.6)
- moved C15 0.54 mm to (95.8, 76.2)
- moved C48 0.48 mm to (147.2, 142.4)
- moved C54 0.48 mm to (71.0, 104.8)
- moved C47 0.43 mm to (282.6, 161.8)
- moved C14 0.42 mm to (313.6, 161.8)
- moved C72 0.41 mm to (99.5, 123.8)
- moved C17 0.36 mm to (80.6, 142.9)
- moved C51 0.35 mm to (280.6, 143.5)
- moved C32 0.35 mm to (333.1, 161.8)
- moved C10 0.35 mm to (94.9, 105.0)
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Routing:
- net +5V: track 359.9 -> 370.5 mm
- net D45: track 319.9 -> 320.6 mm
- net COL1: track 731.6 -> 732.2 mm
- net COL3: track 569.5 -> 570.1 mm

Commit message: changed LEDs fr, added deb to switch
Parts:
- added C23: 0.1uF, Capacitor_SMD:C_0805_2012Metric_Pad1.18x1.45mm_HandSolder, B.Cu at (234.9, 158.1)
- D10, D11, D12, D13, D14, D15, D17, D18, D19, D2, D20, D21, D22, D23, D24, D25, D26, D27, D28, D29, D3, D30, D31, D32, D33, D34, D35, D36, D37, D38, D39, D4, D40, D41, D42, D43, D44, D45, D46, D47, D48, D49, D5, D50, D51, D52, D53, D54, D55, D56, D57, D58, D59, D6, D60, D61, D62, D63, D64, D65, D66, D67, D68, D7, D8, D9: footprint reverse:MX_SK6812MINI-E_REV -> personalLibrary:MX_SK6812MINI-E_REV
- SW16: footprint acheron_MXH:MX200HR -> acheron_MXH:MX200H
- moved C9 11.5 mm to (126.5, 161.8)
- moved C62 11.2 mm to (102.7, 161.8)
- moved C31 10.5 mm to (269.6, 161.6)
- moved C17 10.5 mm to (91.0, 144.3)
- moved C14 10.5 mm to (324.1, 161.8)
- moved C46 10.3 mm to (214.4, 143.1)
- moved C44 10.3 mm to (142.9, 105.0)
- moved C66 10.3 mm to (83.6, 123.9)
- moved C41 10.3 mm to (78.7, 161.8)
- moved C25 10.3 mm to (197.6, 161.8)
- moved C47 10.3 mm to (292.9, 161.9)
- moved C34 10.2 mm to (123.8, 105.3)
- moved C72 10.2 mm to (109.6, 124.1)
- moved C33 10.2 mm to (343.1, 143.3)
- moved C64 10.1 mm to (181.2, 104.8)
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Connections:
- D10 pad 1: Net-(D10-Pad1) -> +5V
- D10 pad 2: GND -> Net-(D10-Pad2)
- D10 pad 3: Net-(D10-Pad3) -> GND
- D10 pad 4: +5V -> Net-(D10-Pad4)
- D11 pad 1: Net-(D11-Pad1) -> +5V
- D11 pad 2: GND -> Net-(D11-Pad2)
- D11 pad 3: Net-(D10-Pad1) -> GND
- D11 pad 4: +5V -> Net-(D10-Pad2)
- D12 pad 1: Net-(D12-Pad1) -> +5V
- D12 pad 2: GND -> Net-(D12-Pad2)
- D12 pad 3: Net-(D11-Pad1) -> GND
- D12 pad 4: +5V -> Net-(D11-Pad2)
- D13 pad 1: Net-(D13-Pad1) -> +5V
- D13 pad 2: GND -> Net-(D13-Pad2)
- D13 pad 3: Net-(D12-Pad1) -> GND
- D13 pad 4: +5V -> Net-(D12-Pad2)
- D14 pad 1: Net-(D14-Pad1) -> +5V
- D14 pad 2: GND -> Net-(D14-Pad2)
- D14 pad 3: Net-(D13-Pad1) -> GND
- D14 pad 4: +5V -> Net-(D13-Pad2)
- D15 pad 1: D16 -> +5V
- D15 pad 2: GND -> D16
- D15 pad 3: Net-(D14-Pad1) -> GND
- D15 pad 4: +5V -> Net-(D14-Pad2)
- D17 pad 1: Net-(D17-Pad1) -> +5V
- D17 pad 2: GND -> Net-(D17-Pad2)
- D17 pad 3: D16 -> GND
- D17 pad 4: +5V -> D16
- D18 pad 1: Net-(D18-Pad1) -> +5V
- D18 pad 2: GND -> Net-(D18-Pad2)
- D18 pad 3: Net-(D17-Pad1) -> GND
- D18 pad 4: +5V -> Net-(D17-Pad2)
- D19 pad 1: Net-(D19-Pad1) -> +5V
- D19 pad 2: GND -> Net-(D19-Pad2)
- D19 pad 3: Net-(D18-Pad1) -> GND
- D19 pad 4: +5V -> Net-(D18-Pad2)
- D2 pad 1: Net-(D2-Pad1) -> +5V
- D2 pad 2: GND -> Net-(D2-Pad2)
- D2 pad 3: LED -> GND
- D2 pad 4: +5V -> LED
- D20 pad 1: Net-(D20-Pad1) -> +5V
- D20 pad 2: GND -> Net-(D20-Pad2)
- D20 pad 3: Net-(D19-Pad1) -> GND
- D20 pad 4: +5V -> Net-(D19-Pad2)
- D21 pad 1: Net-(D21-Pad1) -> +5V
- D21 pad 2: GND -> Net-(D21-Pad2)
- D21 pad 3: Net-(D20-Pad1) -> GND
- D21 pad 4: +5V -> Net-(D20-Pad2)
- D22 pad 1: Net-(D22-Pad1) -> +5V
- D22 pad 2: GND -> Net-(D22-Pad2)
- D22 pad 3: Net-(D21-Pad1) -> GND
- D22 pad 4: +5V -> Net-(D21-Pad2)
- D23 pad 1: Net-(D23-Pad1) -> +5V
- D23 pad 2: GND -> Net-(D23-Pad2)
- D23 pad 3: Net-(D22-Pad1) -> GND
- D23 pad 4: +5V -> Net-(D22-Pad2)
- D24 pad 1: Net-(D24-Pad1) -> +5V
- D24 pad 2: GND -> Net-(D24-Pad2)
- D24 pad 3: Net-(D23-Pad1) -> GND
- D24 pad 4: +5V -> Net-(D23-Pad2)
- D25 pad 1: Net-(D25-Pad1) -> +5V
- D25 pad 2: GND -> Net-(D25-Pad2)
- D25 pad 3: Net-(D24-Pad1) -> GND
- D25 pad 4: +5V -> Net-(D24-Pad2)
- D26 pad 1: Net-(D26-Pad1) -> +5V
- D26 pad 2: GND -> Net-(D26-Pad2)
- D26 pad 3: Net-(D25-Pad1) -> GND
- D26 pad 4: +5V -> Net-(D25-Pad2)
- D27 pad 1: Net-(D27-Pad1) -> +5V
- D27 pad 2: GND -> Net-(D27-Pad2)
- D27 pad 3: Net-(D26-Pad1) -> GND
- D27 pad 4: +5V -> Net-(D26-Pad2)
- D28 pad 1: Net-(D28-Pad1) -> +5V
- D28 pad 2: GND -> Net-(D28-Pad2)
- D28 pad 3: Net-(D27-Pad1) -> GND
- D28 pad 4: +5V -> Net-(D27-Pad2)
- D29 pad 1: Net-(D29-Pad1) -> +5V
- D29 pad 2: GND -> Net-(D29-Pad2)
- D29 pad 3: Net-(D28-Pad1) -> GND
- D29 pad 4: +5V -> Net-(D28-Pad2)
- D3 pad 1: Net-(D3-Pad1) -> +5V
- D3 pad 2: GND -> Net-(D3-Pad2)
- D3 pad 3: Net-(D2-Pad1) -> GND
- D3 pad 4: +5V -> Net-(D2-Pad2)
- D30 pad 1: Net-(D30-Pad1) -> +5V
- D30 pad 2: GND -> Net-(D30-Pad2)
- D30 pad 3: Net-(D29-Pad1) -> GND
- D30 pad 4: +5V -> Net-(D29-Pad2)
- D31 pad 1: D31 -> +5V
- D31 pad 2: GND -> D31
- D31 pad 3: Net-(D30-Pad1) -> GND
- D31 pad 4: +5V -> Net-(D30-Pad2)
- D32 pad 1: Net-(D32-Pad1) -> +5V
- D32 pad 2: GND -> Net-(D32-Pad2)
- D32 pad 3: D31 -> GND
- D32 pad 4: +5V -> D31
- D33 pad 1: Net-(D33-Pad1) -> +5V
- D33 pad 2: GND -> Net-(D33-Pad2)
- D33 pad 3: Net-(D32-Pad1) -> GND
- D33 pad 4: +5V -> Net-(D32-Pad2)
- D34 pad 1: Net-(D34-Pad1) -> +5V
- D34 pad 2: GND -> Net-(D34-Pad2)
- D34 pad 3: Net-(D33-Pad1) -> GND
- D34 pad 4: +5V -> Net-(D33-Pad2)
- D35 pad 1: Net-(D35-Pad1) -> +5V
- D35 pad 2: GND -> Net-(D35-Pad2)
- D35 pad 3: Net-(D34-Pad1) -> GND
- D35 pad 4: +5V -> Net-(D34-Pad2)
- D36 pad 1: Net-(D36-Pad1) -> +5V
- D36 pad 2: GND -> Net-(D36-Pad2)
- D36 pad 3: Net-(D35-Pad1) -> GND
- D36 pad 4: +5V -> Net-(D35-Pad2)
- D37 pad 1: Net-(D37-Pad1) -> +5V
- D37 pad 2: GND -> Net-(D37-Pad2)
- D37 pad 3: Net-(D36-Pad1) -> GND
- D37 pad 4: +5V -> Net-(D36-Pad2)
- D38 pad 1: Net-(D38-Pad1) -> +5V
- D38 pad 2: GND -> Net-(D38-Pad2)
- D38 pad 3: Net-(D37-Pad1) -> GND
- D38 pad 4: +5V -> Net-(D37-Pad2)
- D39 pad 1: Net-(D39-Pad1) -> +5V
- D39 pad 2: GND -> Net-(D39-Pad2)
- D39 pad 3: Net-(D38-Pad1) -> GND
- D39 pad 4: +5V -> Net-(D38-Pad2)
- D4 pad 1: Net-(D4-Pad1) -> +5V
- D4 pad 2: GND -> Net-(D4-Pad2)
- D4 pad 3: Net-(D3-Pad1) -> GND
- D4 pad 4: +5V -> Net-(D3-Pad2)
- D40 pad 1: Net-(D40-Pad1) -> +5V
- D40 pad 2: GND -> Net-(D40-Pad2)
- D40 pad 3: Net-(D39-Pad1) -> GND
- D40 pad 4: +5V -> Net-(D39-Pad2)
- D41 pad 1: Net-(D41-Pad1) -> +5V
- D41 pad 2: GND -> Net-(D41-Pad2)
- D41 pad 3: Net-(D40-Pad1) -> GND
- D41 pad 4: +5V -> Net-(D40-Pad2)
- D42 pad 1: Net-(D42-Pad1) -> +5V
- D42 pad 2: GND -> Net-(D42-Pad2)
- D42 pad 3: Net-(D41-Pad1) -> GND
- D42 pad 4: +5V -> Net-(D41-Pad2)
- D43 pad 1: Net-(D43-Pad1) -> +5V
- D43 pad 2: GND -> Net-(D43-Pad2)
- D43 pad 3: Net-(D42-Pad1) -> GND
- D43 pad 4: +5V -> Net-(D42-Pad2)
- D44 pad 1: Net-(D44-Pad1) -> +5V
- D44 pad 2: GND -> Net-(D44-Pad2)
- D44 pad 3: Net-(D43-Pad1) -> GND
- D44 pad 4: +5V -> Net-(D43-Pad2)
- D45 pad 1: D45 -> +5V
- D45 pad 2: GND -> D45
- D45 pad 3: Net-(D44-Pad1) -> GND
- D45 pad 4: +5V -> Net-(D44-Pad2)
- D46 pad 1: Net-(D46-Pad1) -> +5V
- D46 pad 2: GND -> Net-(D46-Pad2)
- D46 pad 3: D45 -> GND
- D46 pad 4: +5V -> D45
- D47 pad 1: Net-(D47-Pad1) -> +5V
- D47 pad 2: GND -> Net-(D47-Pad2)
- D47 pad 3: Net-(D46-Pad1) -> GND
- D47 pad 4: +5V -> Net-(D46-Pad2)
- D48 pad 1: Net-(D48-Pad1) -> +5V
- D48 pad 2: GND -> Net-(D48-Pad2)
- D48 pad 3: Net-(D47-Pad1) -> GND
- D48 pad 4: +5V -> Net-(D47-Pad2)
- D49 pad 1: Net-(D49-Pad1) -> +5V
- D49 pad 2: GND -> Net-(D49-Pad2)
- D49 pad 3: Net-(D48-Pad1) -> GND
- D49 pad 4: +5V -> Net-(D48-Pad2)
- D5 pad 1: Net-(D5-Pad1) -> +5V
- D5 pad 2: GND -> Net-(D5-Pad2)
- D5 pad 3: Net-(D4-Pad1) -> GND
- D5 pad 4: +5V -> Net-(D4-Pad2)
- D50 pad 1: Net-(D50-Pad1) -> +5V
- D50 pad 2: GND -> Net-(D50-Pad2)
- D50 pad 3: Net-(D49-Pad1) -> GND
- D50 pad 4: +5V -> Net-(D49-Pad2)
- D51 pad 1: Net-(D51-Pad1) -> +5V
- D51 pad 2: GND -> Net-(D51-Pad2)
- D51 pad 3: Net-(D50-Pad1) -> GND
- D51 pad 4: +5V -> Net-(D50-Pad2)
- D52 pad 1: Net-(D52-Pad1) -> +5V
- D52 pad 2: GND -> Net-(D52-Pad2)
- D52 pad 3: Net-(D51-Pad1) -> GND
- D52 pad 4: +5V -> Net-(D51-Pad2)
- D53 pad 1: Net-(D53-Pad1) -> +5V
- D53 pad 2: GND -> Net-(D53-Pad2)
- D53 pad 3: Net-(D52-Pad1) -> GND
- D53 pad 4: +5V -> Net-(D52-Pad2)
- D54 pad 1: Net-(D54-Pad1) -> +5V
- D54 pad 2: GND -> Net-(D54-Pad2)
- D54 pad 3: Net-(D53-Pad1) -> GND
- D54 pad 4: +5V -> Net-(D53-Pad2)
- D55 pad 1: Net-(D55-Pad1) -> +5V
- D55 pad 2: GND -> Net-(D55-Pad2)
- D55 pad 3: Net-(D54-Pad1) -> GND
- D55 pad 4: +5V -> Net-(D54-Pad2)
- D56 pad 1: Net-(D56-Pad1) -> +5V
- D56 pad 2: GND -> Net-(D56-Pad2)
- D56 pad 3: Net-(D55-Pad1) -> GND
- D56 pad 4: +5V -> Net-(D55-Pad2)
- D57 pad 1: Net-(D57-Pad1) -> +5V
- D57 pad 2: GND -> Net-(D57-Pad2)
- D57 pad 3: Net-(D56-Pad1) -> GND
- D57 pad 4: +5V -> Net-(D56-Pad2)
- D58 pad 1: Net-(D58-Pad1) -> +5V
- D58 pad 2: GND -> Net-(D58-Pad2)
- D58 pad 3: Net-(D57-Pad1) -> GND
- D58 pad 4: +5V -> Net-(D57-Pad2)
- D59 pad 1: D59 -> +5V
- D59 pad 2: GND -> D59
- D59 pad 3: Net-(D58-Pad1) -> GND
- D59 pad 4: +5V -> Net-(D58-Pad2)
- D6 pad 1: Net-(D6-Pad1) -> +5V
- D6 pad 2: GND -> Net-(D6-Pad2)
- D6 pad 3: Net-(D5-Pad1) -> GND
- D6 pad 4: +5V -> Net-(D5-Pad2)
- D60 pad 1: Net-(D60-Pad1) -> +5V
- D60 pad 2: GND -> Net-(D60-Pad2)
- D60 pad 3: D59 -> GND
- D60 pad 4: +5V -> D59
- D61 pad 1: Net-(D61-Pad1) -> +5V
- D61 pad 2: GND -> Net-(D61-Pad2)
- D61 pad 3: Net-(D60-Pad1) -> GND
- D61 pad 4: +5V -> Net-(D60-Pad2)
- D62 pad 1: Net-(D62-Pad1) -> +5V
- D62 pad 2: GND -> Net-(D62-Pad2)
- D62 pad 3: Net-(D61-Pad1) -> GND
- D62 pad 4: +5V -> Net-(D61-Pad2)
- D63 pad 1: Net-(D63-Pad1) -> +5V
- D63 pad 2: GND -> Net-(D63-Pad2)
- D63 pad 3: Net-(D62-Pad1) -> GND
- D63 pad 4: +5V -> Net-(D62-Pad2)
- D64 pad 1: Net-(D64-Pad1) -> +5V
- D64 pad 2: GND -> Net-(D64-Pad2)
- D64 pad 3: Net-(D63-Pad1) -> GND
- D64 pad 4: +5V -> Net-(D63-Pad2)
- D65 pad 1: Net-(D65-Pad1) -> +5V
- D65 pad 2: GND -> Net-(D65-Pad2)
- D65 pad 3: Net-(D64-Pad1) -> GND
- D65 pad 4: +5V -> Net-(D64-Pad2)
- D66 pad 1: Net-(D66-Pad1) -> +5V
- D66 pad 2: GND -> Net-(D66-Pad2)
- D66 pad 3: Net-(D65-Pad1) -> GND
- D66 pad 4: +5V -> Net-(D65-Pad2)
- D67 pad 1: Net-(D67-Pad1) -> +5V
- D67 pad 2: GND -> Net-(D67-Pad2)
- D67 pad 3: Net-(D66-Pad1) -> GND
- D67 pad 4: +5V -> Net-(D66-Pad2)
- D68 pad 1: unconnected-(D68-Pad1) -> +5V
- D68 pad 2: GND -> unconnected-(D68-Pad2)
- D68 pad 3: Net-(D67-Pad1) -> GND
- D68 pad 4: +5V -> Net-(D67-Pad2)
- D7 pad 1: Net-(D7-Pad1) -> +5V
- D7 pad 2: GND -> Net-(D7-Pad2)
- D7 pad 3: Net-(D6-Pad1) -> GND
- D7 pad 4: +5V -> Net-(D6-Pad2)
- D8 pad 1: Net-(D8-Pad1) -> +5V
- D8 pad 2: GND -> Net-(D8-Pad2)
- D8 pad 3: Net-(D7-Pad1) -> GND
- D8 pad 4: +5V -> Net-(D7-Pad2)
- D9 pad 1: Net-(D10-Pad3) -> +5V
- D9 pad 2: GND -> Net-(D10-Pad4)
- D9 pad 3: Net-(D8-Pad1) -> GND
- D9 pad 4: +5V -> Net-(D8-Pad2)
- U1 pad 10: MISO -> MOSI
- U1 pad 11: MOSI -> MISO
- U1 pad 12: SCK -> ROW3
- U1 pad 9: ROW3 -> SCK
Routing:
- net D59: track 399.5 -> 13.3 mm, vias 4 -> 0
- net D45: track 320.6 -> 0.04 mm, vias 6 -> 0
- net Net-(D63-Pad2): track 0.00 -> 90.4 mm, vias 0 -> 6
- net +5V: track 370.5 -> 290.8 mm, vias 75 -> 65
- net Net-(D62-Pad2): track 0.00 -> 69.9 mm, vias 0 -> 2
- net Net-(D62-Pad1): track 68.1 -> 0.00 mm, vias 2 -> 0
- net Net-(D63-Pad1): track 67.2 -> 0.00 mm, vias 2 -> 0
- net D31: track 395.5 -> 341.4 mm, vias 12 -> 8
- net GND: track 95.9 -> 54.7 mm, vias 14 -> 7
- net Net-(D3-Pad1): track 32.1 -> 0.00 mm, vias 2 -> 0
- net Net-(D2-Pad1): track 31.5 -> 0.00 mm, vias 2 -> 0
- net Net-(D2-Pad2): track 0.00 -> 30.2 mm, vias 0 -> 2
- net Net-(D46-Pad2): track 0.00 -> 29.4 mm, vias 0 -> 2
- net Net-(D44-Pad2): track 0.00 -> 28.5 mm
- net Net-(D3-Pad2): track 0.00 -> 28.4 mm, vias 0 -> 2
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Other:
- board text removed: "MISO"
- board text removed: "SCK"
