File: keeb.kicad_sch (KiCad schematic)
At the start: 21 parts, among them J1 AVR-ISP-6, SW1 SW_MEC_5E, U1 ATmega32U4-A, Y1 16 Mhz XTAL

Commit message: changed switch, fixed extra capacitor
Parts:
- removed SW1: SW_MEC_5E, Button_Switch_SMD:SW_MEC_5GSH9, symbol Switch:SW_MEC_5E
- added SW1: SW_SPST, Button_Switch_SMD:SW_SPST_TL3342, symbol Switch:SW_SPST
- gave numbers to parts that had none: 1
Connections:
- net GND: now also SW1.1 (A)
- net RESET: now also SW1.2 (B)
Changed lines of the file:
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@@
   (junction (at 46.99 69.85) (diameter 0) (color 0 0 0 0)
   )
-  (junction (at 133.35 125.73) (diameter 0) (color 0 0 0 0)
-  )
   (junction (at 140.97 128.27) (diameter 0) (color 0 0 0 0)
   )
@@
   )
   (junction (at 59.69 38.1) (diameter 0) (color 0 0 0 0)
-  )
-  (junction (at 120.65 125.73) (diameter 0) (color 0 0 0 0)
   )
   (junction (at 44.45 63.5) (diameter 0) (color 0 0 0 0)
@@
     (stroke (width 0) (type default) (color 0 0 0 0))
   )
-  (wire (pts (xy 133.35 123.19) (xy 133.35 125.73))
-    (stroke (width 0) (type default) (color 0 0 0 0))
-  )
   (wire (pts (xy 27.94 172.72) (xy 33.02 172.72))
     (stroke (width 0) (type default) (color 0 0 0 0))
@@
     (stroke (width 0) (type default) (color 0 0 0 0))
   )
-  (wire (pts (xy 120.65 125.73) (xy 120.65 135.89))
+  (wire (pts (xy 120.65 125.73) (xy 120.65 130.81))
     (stroke (width 0) (type default) (color 0 0 0 0))
   )
@@
     (stroke (width 0) (type default) (color 0 0 0 0))
   )
-  (wire (pts (xy 120.65 123.19) (xy 120.65 125.73))
-    (stroke (width 0) (type default) (color 0 0 0 0))
-  )
   (wire (pts (xy 29.21 114.3) (xy 34.29 114.3))
     (stroke (width 0) (type default) (color 0 0 0 0))
@@
     (stroke (width 0) (type default) (color 0 0 0 0))
   )
-  (wire (pts (xy 121.92 123.19) (xy 120.65 123.19))
-    (stroke (width 0) (type default) (color 0 0 0 0))
-  )
   (wire (pts (xy 107.95 158.75) (xy 107.95 157.48))
     (stroke (width 0) (type default) (color 0 0 0 0))
   )
   (wire (pts (xy 43.18 60.96) (xy 46.99 60.96))
-    (stroke (width 0) (type default) (color 0 0 0 0))
-  )
-  (wire (pts (xy 132.08 123.19) (xy 133.35 123.19))
     (stroke (width 0) (type default) (color 0 0 0 0))
   )
@@
     (pin "2")
   )
+  (symbol (lib_id "Switch:SW_SPST") (at 127 125.73 0) (unit 1)
+    (in_bom yes) (on_board yes) (fields_autoplaced)
+    (property "Reference" "SW1" (id 0) (at 127 119.38 0))
+    (property "Value" "SW_SPST" (id 1) (at 127 121.92 0))
+    (property "Footprint" "Button_Switch_SMD:SW_SPST_TL3342" (id 2) (at 127 125.73 0)
+      (effects (font (size 1.27 1.27)) hide)
+    )
+    (property "Datasheet" "~" (id 3) (at 127 125.73 0)
+      (effects (font (size 1.27 1.27)) hide)
+    )
+    (pin "1")
+    (pin "2")
+  )
   (symbol (lib_id "power:+5V") (at 33.02 165.1 0) (unit 1)
     (in_bom yes) (on_board yes) (fields_autoplaced)
@@
   (symbol (lib_id "power:GND") (at 140.97 133.35 0) (unit 1)
     (in_bom yes) (on_board yes)
-    (property "Reference" "#PWR?" (id 0) (at 140.97 139.7 0)
+    (property "Reference" "#PWR0173" (id 0) (at 140.97 139.7 0)
       (effects (font (size 1.27 1.27)) hide)
     )
@@
     (pin "2")
   )
-  (symbol (lib_id "power:GND") (at 120.65 135.89 0) (unit 1)
+  (symbol (lib_id "power:GND") (at 120.65 130.81 0) (unit 1)
     (in_bom yes) (on_board yes)
-    (property "Reference" "#PWR?" (id 0) (at 120.65 142.24 0)
-      (effects (font (size 1.27 1.27)) hide)
-    )
-    (property "Value" "GND" (id 1) (at 118.11 137.16 0)
+    (property "Reference" "#PWR0107" (id 0) (at 120.65 137.16 0)
+      (effects (font (size 1.27 1.27)) hide)
+    )
+    (property "Value" "GND" (id 1) (at 118.11 132.08 0)
       (effects (font (size 0.762 0.762)))
     )
-    (property "Footprint" "" (id 2) (at 120.65 135.89 0)
-      (effects (font (size 1.27 1.27)) hide)
-    )
-    (property "Datasheet" "" (id 3) (at 120.65 135.89 0)
+    (property "Footprint" "" (id 2) (at 120.65 130.81 0)
+      (effects (font (size 1.27 1.27)) hide)
+    )
+    (property "Datasheet" "" (id 3) (at 120.65 130.81 0)
       (effects (font (size 1.27 1.27)) hide)
     )
@@
     (pin "1")
     (pin "2")
-  )
-  (symbol (lib_id "Switch:SW_MEC_5E") (at 127 125.73 0) (unit 1)
-    (in_bom yes) (on_board yes) (fields_autoplaced)
-    (property "Reference" "SW1" (id 0) (at 127 115.57 0))
-    (property "Value" "SW_MEC_5E" (id 1) (at 127 118.11 0))
-    (property "Footprint" "Button_Switch_SMD:SW_MEC_5GSH9" (id 2) (at 127 118.11 0)
-      (effects (font (size 1.27 1.27)) hide)
-    )
-    (property "Datasheet" "http://www.apem.com/int/index.php?controller=attachment&id_attachment=1371" (id 3) (at 127 118.11 0)
-      (effects (font (size 1.27 1.27)) hide)
-    )
-    (pin "1")
-    (pin "2")
-    (pin "3")
-    (pin "4")
   )
   (symbol (lib_id "power:GND") (at 54.61 146.05 0) (unit 1)
@@
   (symbol (lib_id "Device:C_Small") (at 140.97 130.81 0) (unit 1)
     (in_bom yes) (on_board yes) (fields_autoplaced)
-    (property "Reference" "C?" (id 0) (at 143.51 129.5462 0)
+    (property "Reference" "C23" (id 0) (at 143.51 129.5462 0)
       (effects (font (size 1.27 1.27)) (justify left))
     )
@@
       (reference "#PWR0106") (unit 1) (value "GND") (footprint "")
     )
+    (path "/4b67369c-c799-42f6-88d7-4748c635b2b6"
+      (reference "#PWR0107") (unit 1) (value "GND") (footprint "")
+    )
     (path "/62c2bd71-a0c6-4ae9-936e-1116afe2ff6f"
       (reference "#PWR0108") (unit 1) (value "GND") (footprint "")
@@
       (reference "#PWR0172") (unit 1) (value "GND") (footprint "")
     )
+    (path "/2f1b12c4-f7a9-4eb2-b8af-faf54ae9b755"
+      (reference "#PWR0173") (unit 1) (value "GND") (footprint "")
+    )
     (path "/40940281-55a3-43d0-8f01-7316aa0f04ca/605f7b62-a00b-4afb-a74f-e86a2747d377"
       (reference "#PWR0174") (unit 1) (value "GND") (footprint "")
@@
       (reference "#PWR0205") (unit 1) (value "GND") (footprint "")
     )
-    (path "/2f1b12c4-f7a9-4eb2-b8af-faf54ae9b755"
-      (reference "#PWR?") (unit 1) (value "GND") (footprint "")
-    )
-    (path "/4b67369c-c799-42f6-88d7-4748c635b2b6"
-      (reference "#PWR?") (unit 1) (value "GND") (footprint "")
-    )
     (path "/2c94f5c9-ba82-4e7b-993f-ef5397d3358f"
       (reference "C1") (unit 1) (value "22pF") (footprint "Capacitor_SMD:C_0805_2012Metric_Pad1.18x1.45mm_HandSolder")
@@
       (reference "C22") (unit 1) (value "100nF") (footprint "Capacitor_SMD:C_0805_2012Metric_Pad1.18x1.45mm_HandSolder")
     )
+    (path "/d0c216ff-9a53-4ff8-83b4-43ebcf388166"
+      (reference "C23") (unit 1) (value "0.1uF") (footprint "Capacitor_SMD:C_0805_2012Metric_Pad1.18x1.45mm_HandSolder")
+    )
     (path "/40940281-55a3-43d0-8f01-7316aa0f04ca/b3d146f1-8098-4d85-b28c-4292e494c7b1"
       (reference "C24") (unit 1) (value "100nF") (footprint "Capacitor_SMD:C_0805_2012Metric_Pad1.18x1.45mm_HandSolder")
@@
       (reference "C75") (unit 1) (value "100nF") (footprint "Capacitor_SMD:C_0805_2012Metric_Pad1.18x1.45mm_HandSolder")
     )
-    (path "/d0c216ff-9a53-4ff8-83b4-43ebcf388166"
-      (reference "C?") (unit 1) (value "0.1uF") (footprint "Capacitor_SMD:C_0805_2012Metric_Pad1.18x1.45mm_HandSolder")
-    )
     (path "/e9764993-7462-40fd-8d4b-02d010ee99fe"
       (reference "D1") (unit 1) (value "PRTR5V0U2X") (footprint "random-keyboard-parts2:SOT143B")
@@
       (reference "R6") (unit 1) (value "10k") (footprint "Resistor_SMD:R_0805_2012Metric_Pad1.20x1.40mm_HandSolder")
     )
-    (path "/9d0ee07a-506a-41bd-81ab-8b5fbd38bdf0"
-      (reference "SW1") (unit 1) (value "SW_MEC_5E") (footprint "Button_Switch_SMD:SW_MEC_5GSH9")
+    (path "/1e3f6d33-9a3c-48e7-8087-e739cff5ef01"
+      (reference "SW1") (unit 1) (value "SW_SPST") (footprint "Button_Switch_SMD:SW_SPST_TL3342")
     )
     (path "/39dabec8-ee69-4816-aadc-d8efa99bb3bd/de0d3458-7d32-4758-ae71-7f9dc1a93c97"
